File: home_automation.kicad_pcb (KiCad board)
At the start: 2 copper layers, 48 parts, among them J1 AC In, J2 NodeMCU Header, J3 NodeMCU Header, J4 SW_4, J5 DHT11, J6 SW_1, J7 SW_3, J8 SW_2, K1 Relay_SPDT, K2 Relay_SPDT, K3 Relay_SPDT, K4 Relay_SPDT, Q1 D882, Q2 D882, Q3 D882, Q4 D882, SW1 SW_DIP_x02, SW2 SW_DIP_x02, SW3 SW_DIP_x02, SW4 SW_DIP_x02, U1 PC817, U2 PC817, U3 LM7805_TO220, U4 PC817, U5 PC817, U6 NodeMCU

Commit message: Placing and Back layer wiring
Parts:
- J1: value AC In -> AC_in; footprint Connector_PinHeader_2.54mm:PinHeader_1x02_P2.54mm_Vertical -> TerminalBlock:TerminalBlock_bornier-2_P5.08mm
- J4: value SW_4 -> Sw_1; footprint Connector_Phoenix_MSTB:PhoenixContact_MSTBA_2,5_3-G_1x03_P5.00mm_Horizontal -> TerminalBlock:TerminalBlock_bornier-3_P5.08mm
- J6: value SW_1 -> Sw_2; footprint Connector_Phoenix_MSTB:PhoenixContact_MSTBA_2,5_3-G_1x03_P5.00mm_Horizontal -> TerminalBlock:TerminalBlock_bornier-3_P5.08mm
- J7: value SW_3 -> Sw_3; footprint Connector_Phoenix_MSTB:PhoenixContact_MSTBA_2,5_3-G_1x03_P5.00mm_Horizontal -> TerminalBlock:TerminalBlock_bornier-3_P5.08mm
- J8: value SW_2 -> Sw_4; footprint Connector_Phoenix_MSTB:PhoenixContact_MSTBA_2,5_3-G_1x03_P5.00mm_Horizontal -> TerminalBlock:TerminalBlock_bornier-3_P5.08mm
- R1, R2, R3, R4, R5: footprint Resistor_THT:R_Axial_DIN0414_L11.9mm_D4.5mm_P15.24mm_Horizontal -> Resistor_THT:R_Axial_DIN0309_L9.0mm_D3.2mm_P12.70mm_Horizontal
- R10, R6, R7, R9: footprint Resistor_THT:R_Axial_DIN0516_L15.5mm_D5.0mm_P25.40mm_Horizontal -> Resistor_THT:R_Axial_DIN0309_L9.0mm_D3.2mm_P12.70mm_Horizontal
- R8: footprint Resistor_THT:R_Axial_DIN0516_L15.5mm_D5.0mm_P25.40mm_Horizontal -> Resistor_THT:R_Axial_DIN0414_L11.9mm_D4.5mm_P15.24mm_Horizontal
- moved D6 349.0 mm to (101.7, 147.2)
- moved D8 331.0 mm to (108.5, 147.4)
- moved D2 327.1 mm to (87.8, 147.1)
- moved J6 318.4 mm to (87.5, 115.7), turned to 90 degrees
- moved J1 316.3 mm to (89.6, 55.7), turned to 90 degrees
- moved R1 314.1 mm to (89.4, 128.4), turned to -90 degrees
- moved D3 310.0 mm to (94.5, 147.1)
- moved U2 303.5 mm to (124.5, 105.6)
- moved J4 299.4 mm to (86.8, 86.6), turned to 90 degrees
- moved R2 288.2 mm to (96.0, 128.4), turned to -90 degrees
- moved K1 286.7 mm to (103.2, 81.7), turned to 180 degrees
- moved C1 286.1 mm to (143.6, 54.0), turned to -90 degrees
- moved U1 286.0 mm to (120.8, 74.9)
- moved K2 283.6 mm to (103.1, 110.7), turned to 180 degrees
- moved J5 282.6 mm to (181.0, 47.6), turned to 90 degrees
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Connections:
- net Net-(J2-Pad1) renamed /A0
- net Net-(J2-Pad11) renamed /3V3-1
- net Net-(J2-Pad12) renamed /EN
- net Net-(J2-Pad13) renamed /RST
- net Net-(J2-Pad2) renamed /RSV1
- net Net-(J2-Pad3) renamed /RSV2
- net Net-(J2-Pad4) renamed /SD3
- net Net-(J2-Pad5) renamed /SD2
- net Net-(J2-Pad6) renamed /SD1
- net Net-(J2-Pad7) renamed /CMD
- net Net-(J2-Pad8) renamed /SD0
- net Net-(J2-Pad9) renamed /CLK
- net Net-(J3-Pad12) renamed /RX
- net Net-(J3-Pad13) renamed /TX
- net Net-(J3-Pad15) renamed /3V3-2
- net Net-(J3-Pad6) renamed /3v3-3
- J1 pad 1: /L -> /N
- J1 pad 2: /N -> /L
- J4 pad 3: /NO_4 -> /NO
- J6 pad 3: /NO -> /NO_2
- J8 pad 3: /NO_2 -> /NO_4
Routing:
- net /12v: track 0.00 -> 229.9 mm
- net /N: track 0.00 -> 217.0 mm
- net /L: track 0.00 -> 214.0 mm
- net GND: track 0.00 -> 151.8 mm
- net /5v: track 0.00 -> 79.1 mm
- net /3V3-1: track 0.00 -> 51.5 mm
- net Net-(R10-Pad1): track 0.00 -> 27.0 mm
- net Net-(R6-Pad1): track 0.00 -> 24.9 mm
- net Net-(R9-Pad1): track 0.00 -> 22.6 mm
- net Net-(R7-Pad1): track 0.00 -> 16.7 mm
- net /D7: track 0.00 -> 16.7 mm
- net /D8: track 0.00 -> 16.7 mm
- net /D6: track 0.00 -> 16.7 mm
- net /D5: track 0.00 -> 16.7 mm
- net /Base_2: track 0.00 -> 15.0 mm
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
Commit message: Routing Completed
Parts:
- added REF**: MountingHole_2.5mm_Pad_Via, MountingHole:MountingHole_2.5mm_Pad_Via, F.Cu at (211.2, 43.2)
- added REF**: MountingHole_2.5mm_Pad_Via, MountingHole:MountingHole_2.5mm_Pad_Via, F.Cu at (83.5, 43.6)
- added REF**: MountingHole_2.5mm_Pad_Via, MountingHole:MountingHole_2.5mm_Pad_Via, F.Cu at (211.1, 150.6)
- added REF**: MountingHole_2.5mm_Pad_Via, MountingHole:MountingHole_2.5mm_Pad_Via, F.Cu at (83.3, 150.6)
- added REF**: ESD-Logo_8.9x8mm_SilkScreen, Symbol:ESD-Logo_8.9x8mm_SilkScreen, B.Cu at (97.0, 52.6)
- added REF**: KiCad-Logo2_6mm_SilkScreen, Symbol:KiCad-Logo2_6mm_SilkScreen, B.Cu at (199.9, 130.7)
- added REF**: OSHW-Logo2_14.6x12mm_SilkScreen, Symbol:OSHW-Logo2_14.6x12mm_SilkScreen, B.Cu at (96.3, 134.9)
- K1, K2, K3, K4: value Relay_SPDT -> 12V Relay
- U3: value LM7805_TO220 -> LM7805
- moved D5 0.34 mm to (150.2, 116.5)
- moved R2 0.29 mm to (96.3, 128.4)
- moved U6 0.17 mm to (160.1, 87.7)
Routing:
- net GND: track 151.8 -> 566.4 mm, vias 0 -> 9
- net Net-(R1-Pad1): track 0.00 -> 91.8 mm
- net /D5: track 16.7 -> 106.7 mm, vias 0 -> 4
- net /D1: track 4.15 -> 88.7 mm, vias 0 -> 6
- net /D2: track 4.15 -> 88.3 mm, vias 0 -> 4
- net Net-(R5-Pad1): track 0.00 -> 78.5 mm
- net /D7: track 16.7 -> 90.9 mm, vias 0 -> 6
- net /D6: track 16.7 -> 88.1 mm, vias 0 -> 4
- net /D3: track 4.15 -> 74.4 mm, vias 0 -> 3
- net /D8: track 16.7 -> 86.9 mm, vias 0 -> 4
- net Net-(R3-Pad1): track 0.00 -> 53.6 mm
- net /D0: track 14.3 -> 65.1 mm
- net Net-(R2-Pad1): track 0.00 -> 42.1 mm
- net /Collector_2: track 9.89 -> 37.1 mm, vias 0 -> 2
- net /Collector_3: track 6.68 -> 28.6 mm
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- added copper zone on B.Cu, net /3V3-1
- added copper zone on F.Cu, net GND
Other:
- board outline added: 135 x 114.2 mm
- board text added: "Home Automation And Temperature Sensor"
- board text added: "L"
- board text added: "N"
- board text added: "Switch 1"
- board text added: "Switch 2"
- board text added: "Switch 3"
- board text added: "Switch 4"
- board text added: "X"
